File: as3320_BP/as3320-Bandpass.sch (EAGLE design)
At the start: 55 parts, among them IC1 TL074D, IC2 CEM3320, IC3 LM4040 5.0V, IC4 TL074D

Commit message: updated readme
Other:
- note added: "Based on : https://github.com/forestcaver/Analog-Voice/tree/master/AJH_as3320_LPF By Forest Caver CC-BY-NC-SA 4.0"
- note removed: "Based on : https://github.com/acobley/Analog-Voice By Forest Caver CC-BY-NC-SA 4.0"
Changed lines of the file:
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@@
 <setting verticaltext="up"/>
 </settings>
-<grid distance="0.01" unitdist="inch" unit="inch" style="lines" multiple="1" display="no" altdistance="0.01" altunitdist="inch" altunit="inch"/>
+<grid distance="0.1" unitdist="inch" unit="inch" style="lines" multiple="1" display="no" altdistance="0.01" altunitdist="inch" altunit="inch"/>
 <layers>
 <layer number="1" name="Top" color="4" fill="1" visible="no" active="no"/>
@@
 <text x="-31.496" y="-29.718" size="1.778" layer="91">See note in resonance section on possible values for R25</text>
 <text x="-146.05" y="-68.072" size="1.778" layer="91">Based on :
-https://github.com/acobley/Analog-Voice
+https://github.com/forestcaver/Analog-Voice/tree/master/AJH_as3320_LPF
 By  Forest Caver
 CC-BY-NC-SA 4.0</text>
