File: as3320-Vowel/as3320-Vowel-1.brd (EAGLE design)
At the start: 92 x 128.6 mm, 136 parts, among them IC1 TL074D, IC2 CEM3320, IC3 LM4040 5.0V, IC4 TL074D, IC5 CEM3320, IC6 CEM3320, IC7 TL074D, IC9 TL074D

Commit message: Updated to resonance voltage control
Parts:
- removed IN1POT, IN1POT1, IN1POT2: 100K, GMSN:POT
- added C25, C26, C27, C28, C29, C30, C31, C32: 100n, rcl:C0805K
- added D5, D6, D8: 5.1V, diode:SOT23
- added D7: 1N4001, GMSN:SMADIODE
- added IN1LEVEL, IN2LEVEL, IN3LEVEL: 100K, GMSN:POT
- added RES-2, RES-3: PJ301_THONKICONN6, og-pj301_variations:WQP_PJ_301M6
- C1, C15, C16, C17, C19, C2, C20, C21, C22, C3, C4, C5, C6, C7, C8, C9: device rcl:C0603 -> rcl:C0805K
- C10, C24: device rcl:C0603 -> Pure VCF:GMSN_C0805K
- C11: device rcl:C0603 -> Pure VCF:GMSN_M0805
- D3, D4: value 1N5819HW -> 1N4001; device diode:SOD123 -> GMSN:SMADIODE
- POWER: value (none) -> SMD
- R1, R4: device rcl:R0805 -> Pure VCF:GMSN_M0805
- R10, R11, R2, R23, R28, R29, R3, R31, R32, R34, R35, R57, R58, R59, R6, R61, R63, R64, R65, R66, R68, R7, R8: device resistor:R0603 -> Pure VCF:GMSN_M0805
- R12, R13, R14, R15, R16, R17, R18, R19, R20, R21, R22, R24, R25, R26, R27, R30, R33, R36, R37, R38, R39, R40, R41, R42, R43, R44, R45, R46, R47, R48, R49, R50, R51, R52, R53, R54: device rcl:R0603 -> Pure VCF:GMSN_M0805
- R5: device GMSN:R0805 -> Pure VCF:GMSN_M0805
- R70, R72: value 10k -> 100k; device GMSN:R0805 -> Pure VCF:GMSN_M0805
- R71: value 10k -> 100k
- R73, R74: value 5k -> 100k
- moved D4 209.3 mm to (-79.0, 30.0)
- moved R57 198.2 mm to (-116.7, 10.8)
- moved R58 194.7 mm to (-114.7, -9.43)
- moved R74 192.2 mm to (-80.0, -3.00)
- moved R72 183.1 mm to (-80.0, 17.0)
- moved D3 181.7 mm to (-79.0, 10.0)
- moved R70 179.4 mm to (-80.0, 23.0)
- moved RES-1 177.3 mm to (-90.0, 40.0), flipped to the bottom
- moved R73 176.9 mm to (-94.0, -9.00)
- moved C17 175.9 mm to (-113.0, 55.0)
- moved R69 175.0 mm to (-94.0, 29.0)
- moved R39 172.7 mm to (-116.0, 46.0)
- moved D1 172.0 mm to (-116.9, 87.9), turned to 90 degrees
- moved R40 168.9 mm to (-116.0, 41.0)
- moved R71 166.6 mm to (-94.0, 10.0)
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Connections:
- removed net 10V1: IC9.3, RES-1.P3
- removed net N$20: D2.C, POWER.2
- new net -12V-P: D2.C, POWER.1, POWER.2
- new net N$91: D7.A, RES-3.P3
- new net N$92: D7.C, R74.2
- new net N$93: D8.3, IC1.13, R74.1
- net -12V: now also C26.2, C28.2, C30.2, C32.2
- net 10V: no longer R69.2
- net 12V: now also C25.1, C27.1, C29.1, C31.1
- net 5V: now also R69.2, R71.2, R73.2
- net GND: now also C25.2, C26.1, C27.2, C28.1, C29.2, C30.1, C31.2, C32.1, D5.1, D6.1, D8.1, IN1LEVEL.P$1, IN2LEVEL.P$1, IN3LEVEL.P$1, RES-2.P1, RES-3.P1; no longer IC9.10, IC9.12, IN1POT.P$1, IN1POT1.P$1, IN1POT2.P$1
- net N$6: now also POWER.9
- net N$76: now also IN1LEVEL.P$3; no longer IN1POT.P$3
- net N$77: now also IN2LEVEL.P$3; no longer IN1POT1.P$3
- net N$78: now also D3.A, RES-2.P3; no longer POWER.1
- net N$79: now also IN1LEVEL.P$2; no longer IN1POT.P$2
- net N$80: now also IN2LEVEL.P$2; no longer IN1POT1.P$2
- net N$82: now also IN3LEVEL.P$3; no longer IN1POT2.P$3
- net N$83: now also IN3LEVEL.P$2; no longer IN1POT2.P$2
- net N$85: now also D3.C; no longer IC9.1, IC9.2, R70.1
- net N$86: now also D4.A, RES-1.P3; no longer D3.C, IC9.9, R70.2, R71.2
- net N$87: now also R70.2; no longer D3.A, IC9.8
- net N$88: now also D5.3, IC9.3, R70.1; no longer D4.A, R71.1, R73.2
- net N$89: now also D6.3, IC9.10; no longer IC9.13, R73.1, R74.2
- net N$9: now also R71.1, RES-2.P2; no longer POWER.9
- net N$90: now also R73.1, RES-3.P2; no longer IC9.14, R74.1
- net RESONANCE_IN1: now also IC9.1, IC9.2
- net RESONANCE_IN2: now also IC9.8, IC9.9
- net RESONANCE_IN3: now also IC1.12, IC1.14
Routing:
- net GND: track 0.00 -> 833.4 mm, vias 0 -> 8
- net -12V: track 0.00 -> 460.3 mm, vias 0 -> 10
- net 12V: track 0.00 -> 326.8 mm, vias 0 -> 10
- net 5V: track 0.00 -> 247.6 mm, vias 0 -> 1
- net -5V: track 0.00 -> 205.6 mm, vias 0 -> 5
- net RESONANCE_IN2: track 0.00 -> 168.4 mm, vias 0 -> 6
- net N$89: track 0.00 -> 167.2 mm, vias 0 -> 2
- net 10V: track 0.00 -> 159.3 mm, vias 0 -> 4
- net N$3: track 0.00 -> 129.3 mm, vias 0 -> 2
- net BANDPASS_IN: track 0.00 -> 120.8 mm, vias 0 -> 6
- net N$71: track 0.00 -> 106.2 mm, vias 0 -> 2
- net FREQ_IN2: track 0.00 -> 102.5 mm, vias 0 -> 4
- net -5VIN: track 0.00 -> 99.8 mm, vias 0 -> 2
- net N$12: track 0.00 -> 98.6 mm, vias 0 -> 3
- net BANDPASS_OUT1: track 0.00 -> 95.2 mm, vias 0 -> 4
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Other:
- board size 92 x 128.6 mm -> 111.4 x 128.6 mm
- board text added: "-12V"
- board text added: "Inputs"
- board text added: "Triple band pass filter Design Andy C"
- board text removed: "CV1"
- board text removed: "Reset"
- board text removed: "Sequencer Design Andy C"
- board text removed: "Start"
- board text removed: "Tempo"
- board text removed: "Trig 1b"

Commit message: fixed resonance input routing
Connections:
- new net RESONANCE_CTL1: R25.2, R4-RES1.P$2
- new net RESONANCE_CTL2: R39.2, R55-RES2.P$2
- new net RESONANCE_CTL3: R51.2, R56-RES3.P$2
- net 5V: no longer R4-RES1.P$1, R55-RES2.P$1, R56-RES3.P$1
- net RESONANCE_IN1: now also R4-RES1.P$1; no longer R25.2, R4-RES1.P$2
- net RESONANCE_IN2: now also R55-RES2.P$1; no longer R39.2, R55-RES2.P$2
- net RESONANCE_IN3: now also R56-RES3.P$1; no longer R51.2, R56-RES3.P$2
Routing:
- net 5V: track 247.6 -> 225.1 mm
- net RESONANCE_IN3: track 57.3 -> 79.1 mm
- net RESONANCE_IN1: track 91.9 -> 74.3 mm
- net RESONANCE_CTL1: track 0.00 -> 17.5 mm
Changed lines of the file:
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@@
 <drawing>
 <settings>
-<setting alwaysvectorfont="yes"/>
+<setting alwaysvectorfont="no"/>
 <setting verticaltext="up"/>
 </settings>
@@
 <signal name="5V" class="1">
 <contactref element="R32" pad="2"/>
-<contactref element="R4-RES1" pad="P$1"/>
 <contactref element="IC4" pad="8"/>
-<contactref element="R55-RES2" pad="P$1"/>
-<contactref element="R56-RES3" pad="P$1"/>
 <contactref element="R69" pad="2"/>
 <contactref element="R71" pad="2"/>
@@
 <wire x1="-92.964" y1="-8.9408" x2="-93.05" y2="-9" width="0.4064" layer="1"/>
 <wire x1="-92.964" y1="9.9568" x2="-93.05" y2="10" width="0.4064" layer="1"/>
-<wire x1="-67.4624" y1="-0.9144" x2="-67.4624" y2="-6.604" width="0.4064" layer="16"/>
-<wire x1="-64.9224" y1="1.6256" x2="-67.4624" y2="-0.9144" width="0.4064" layer="16"/>
-<wire x1="-64.9224" y1="10.668" x2="-64.9224" y2="1.6256" width="0.4064" layer="16"/>
-<wire x1="-67.4624" y1="13.208" x2="-64.9224" y2="10.668" width="0.4064" layer="16"/>
-<wire x1="-67.4624" y1="-6.604" x2="-67.5" y2="-6.7" width="0.4064" layer="16"/>
-<wire x1="-67.4624" y1="13.208" x2="-67.5" y2="13.3" width="0.4064" layer="16"/>
 <wire x1="-74.4728" y1="7.7216" x2="-92.964" y2="7.7216" width="0.4064" layer="1"/>
 <wire x1="-68.9864" y1="13.208" x2="-74.4728" y2="7.7216" width="0.4064" layer="1"/>
 <wire x1="-67.564" y1="13.208" x2="-68.9864" y2="13.208" width="0.4064" layer="1"/>
-<wire x1="-67.564" y1="13.208" x2="-67.5" y2="13.3" width="0.4064" layer="1"/>
 <wire x1="-80.0608" y1="93.8784" x2="-83.9216" y2="93.8784" width="0.4064" layer="1"/>
 <wire x1="-77.9272" y1="96.012" x2="-80.0608" y2="93.8784" width="0.4064" layer="1"/>
@@
 <wire x1="-71.4248" y1="29.3624" x2="-71.7296" y2="29.0576" width="0.4064" layer="16"/>
 <wire x1="-92.964" y1="29.0576" x2="-93.05" y2="29" width="0.4064" layer="1"/>
-<wire x1="-67.564" y1="33.2232" x2="-67.5" y2="33.3" width="0.4064" layer="16"/>
 <wire x1="-90.0176" y1="100.2792" x2="-87.7824" y2="98.044" width="0.4064" layer="1"/>
 <wire x1="-103.632" y1="100.2792" x2="-90.0176" y2="100.2792" width="0.4064" layer="1"/>
@@
 <wire x1="-79.3496" y1="33.3248" x2="-87.376" y2="41.3512" width="0.4064" layer="1"/>
 <wire x1="-67.564" y1="33.3248" x2="-79.3496" y2="33.3248" width="0.4064" layer="1"/>
-<wire x1="-67.564" y1="33.3248" x2="-67.5" y2="33.3" width="0.4064" layer="1"/>
 <wire x1="-67.3608" y1="19.9136" x2="-67.3608" y2="13.4112" width="0.4064" layer="16"/>
 <wire x1="-65.024" y1="22.2504" x2="-67.3608" y2="19.9136" width="0.4064" layer="16"/>
 <wire x1="-65.024" y1="22.9616" x2="-65.024" y2="22.2504" width="0.4064" layer="16"/>
 <wire x1="-71.4248" y1="29.3624" x2="-65.024" y2="22.9616" width="0.4064" layer="16"/>
-<wire x1="-67.3608" y1="13.4112" x2="-67.5" y2="13.3" width="0.4064" layer="16"/>
 <via x="-88.1888" y="29.0576" extent="1-16" drill="0.4"/>
+<wire x1="-67.3608" y1="13.4112" x2="-67.564" y2="13.208" width="0" layer="19" extent="1-16"/>
+<wire x1="-67.564" y1="33.3248" x2="-67.564" y2="33.2232" width="0" layer="19" extent="1-16"/>
 </signal>
 <signal name="-5V" class="1">
@@
 </signal>
 <signal name="RESONANCE_IN1">
-<contactref element="R25" pad="2"/>
-<contactref element="R4-RES1" pad="P$2"/>
 <contactref element="IC9" pad="1"/>
 <contactref element="IC9" pad="2"/>
@@
 <wire x1="-69.7992" y1="92.456" x2="-69.81" y2="92.4" width="0.2032" layer="1"/>
 <wire x1="-68.58" y1="92.456" x2="-68.54" y2="92.4" width="0.2032" layer="1"/>
-<wire x1="-80.0608" y1="36.1696" x2="-80.8736" y2="36.9824" width="0.2032" layer="1"/>
-<wire x1="-80.0608" y1="36.068" x2="-80.0608" y2="36.1696" width="0.2032" layer="1"/>
-<wire x1="-78.6384" y1="34.6456" x2="-80.0608" y2="36.068" width="0.2032" layer="1"/>
-<wire x1="-66.3448" y1="34.6456" x2="-78.6384" y2="34.6456" width="0.2032" layer="1"/>
-<wire x1="-65.024" y1="33.3248" x2="-66.3448" y2="34.6456" width="0.2032" layer="1"/>
-<wire x1="-80.8736" y1="36.9824" x2="-80.95" y2="37" width="0.2032" layer="1"/>
-<wire x1="-65.024" y1="33.3248" x2="-65" y2="33.3" width="0.2032" layer="1"/>
 <wire x1="-71.628" y1="92.3544" x2="-69.9008" y2="92.3544" width="0.2032" layer="1"/>
 <wire x1="-74.9808" y1="89.0016" x2="-71.628" y2="92.3544" width="0.2032" layer="1"/>
@@
 <wire x1="-80.9752" y1="37.084" x2="-86.868" y2="42.9768" width="0.2032" layer="1"/>
 <wire x1="-69.9008" y1="92.3544" x2="-69.81" y2="92.4" width="0.2032" layer="1"/>
-<wire x1="-80.9752" y1="37.084" x2="-80.95" y2="37" width="0.2032" layer="1"/>
 <via x="-81.1784" y="83.2104" extent="1-16" drill="0.4"/>
 <via x="-93.7768" y="64.008" extent="1-16" drill="0.4"/>
+<contactref element="R4-RES1" pad="P$1"/>
+<wire x1="-80.9752" y1="37.084" x2="-67.5" y2="33.3" width="0" layer="19" extent="1-1"/>
 </signal>
 <signal name="RESONANCE_IN2">
-<contactref element="R39" pad="2"/>
-<contactref element="R55-RES2" pad="P$2"/>
 <contactref element="IC9" pad="8"/>
 <contactref element="IC9" pad="9"/>
@@
 <wire x1="-66.3448" y1="14.6304" x2="-66.7512" y2="14.6304" width="0.2032" layer="1"/>
 <wire x1="-65.024" y1="13.3096" x2="-66.3448" y2="14.6304" width="0.2032" layer="1"/>
-<wire x1="-115.0112" y1="45.9232" x2="-115.05" y2="46" width="0.2032" layer="1"/>
-<wire x1="-65.024" y1="13.3096" x2="-65" y2="13.3" width="0.2032" layer="1"/>
 <wire x1="-63.3984" y1="98.1456" x2="-63.3984" y2="97.7392" width="0.2032" layer="1"/>
 <wire x1="-66.04" y1="100.7872" x2="-63.3984" y2="98.1456" width="0.2032" layer="1"/>
@@
 <via x="-106.4768" y="82.296" extent="1-16" drill="0.4"/>
 <via x="-112.1664" y="60.7568" extent="1-16" drill="0.4"/>
+<contactref element="R55-RES2" pad="P$1"/>
+<wire x1="-65.024" y1="13.3096" x2="-67.5" y2="13.3" width="0" layer="19" extent="1-1"/>
 </signal>
 <signal name="RESONANCE_IN3">
-<contactref element="R51" pad="2"/>
-<contactref element="R56-RES3" pad="P$2"/>
 <contactref element="IC1" pad="14"/>
 <contactref element="IC1" pad="12"/>
@@
 <wire x1="-46.8376" y1="16.1544" x2="-48.0568" y2="16.1544" width="0.2032" layer="1"/>
 <wire x1="-46.3296" y1="15.6464" x2="-46.8376" y2="16.1544" width="0.2032" layer="1"/>
-<wire x1="-53.0352" y1="32.9184" x2="-53.05" y2="33" width="0.2032" layer="1"/>
 <wire x1="-46.3296" y1="15.6464" x2="-46.309" y2="15.602" width="0.2032" layer="1"/>
 <wire x1="-45.6184" y1="13.1064" x2="-46.228" y2="13.1064" width="0.2032" layer="1"/>
@@
 <wire x1="-46.9392" y1="13.0048" x2="-48.6664" y2="11.2776" width="0.2032" layer="1"/>
 <wire x1="-46.3296" y1="13.0048" x2="-46.9392" y2="13.0048" width="0.2032" layer="1"/>
-<wire x1="-64.9224" y1="-6.7056" x2="-65" y2="-6.7" width="0.2032" layer="1"/>
 <wire x1="-46.3296" y1="13.0048" x2="-46.309" y2="13.062" width="0.2032" layer="1"/>
 <via x="-53.0352" y="26.5176" extent="1-16" drill="0.4"/>
 <via x="-48.0568" y="16.1544" extent="1-16" drill="0.4"/>
+<contactref element="R56-RES3" pad="P$1"/>
+<wire x1="-67.4624" y1="-0.9144" x2="-67.4624" y2="-6.604" width="0.4064" layer="16"/>
+<wire x1="-64.9224" y1="1.6256" x2="-67.4624" y2="-0.9144" width="0.4064" layer="16"/>
+<wire x1="-64.9224" y1="10.668" x2="-64.9224" y2="1.6256" width="0.4064" layer="16"/>
+<wire x1="-67.4624" y1="13.208" x2="-64.9224" y2="10.668" width="0.4064" layer="16"/>
+<wire x1="-67.4624" y1="-6.604" x2="-67.5" y2="-6.7" width="0.4064" layer="16"/>
+<wire x1="-64.9224" y1="-6.7056" x2="-67.5" y2="-6.7" width="0" layer="19" extent="1-1"/>
 </signal>
 <signal name="FREQ_IN1">
@@
 <wire x1="-84.1248" y1="51.1048" x2="-84.16" y2="51.19" width="0.2032" layer="1"/>
 </signal>
+<signal name="RESONANCE_CTL1">
+<contactref element="R25" pad="2"/>
+<contactref element="R4-RES1" pad="P$2"/>
+<wire x1="-80.0608" y1="36.1696" x2="-80.8736" y2="36.9824" width="0.2032" layer="1"/>
+<wire x1="-80.0608" y1="36.068" x2="-80.0608" y2="36.1696" width="0.2032" layer="1"/>
+<wire x1="-78.6384" y1="34.6456" x2="-80.0608" y2="36.068" width="0.2032" layer="1"/>
+<wire x1="-66.3448" y1="34.6456" x2="-78.6384" y2="34.6456" width="0.2032" layer="1"/>
+<wire x1="-65.024" y1="33.3248" x2="-66.3448" y2="34.6456" width="0.2032" layer="1"/>
+<wire x1="-65.024" y1="33.3248" x2="-65" y2="33.3" width="0.2032" layer="1"/>
+<wire x1="-80.8736" y1="36.9824" x2="-80.95" y2="37" width="0" layer="19" extent="1-1"/>
+</signal>
+<signal name="RESONANCE_CTL3">
+<contactref element="R51" pad="2"/>
+<contactref element="R56-RES3" pad="P$2"/>
+<wire x1="-53.05" y1="33" x2="-65" y2="-6.7" width="0" layer="19" extent="1-1"/>
+</signal>
+<signal name="RESONANCE_CTL2">
+<contactref element="R39" pad="2"/>
+<contactref element="R55-RES2" pad="P$2"/>
+<wire x1="-65" y1="13.3" x2="-115.05" y2="46" width="0" layer="19" extent="1-1"/>
+</signal>
 </signals>
