File: as3320-Vowel/as3320-Vowel-1.sch (EAGLE design)
At the start: 132 parts, among them IC1 TL074D, IC2 CEM3320, IC3 LM4040 5.0V, IC4 TL074D, IC5 CEM3320, IC6 CEM3320, IC7 TL074D, IC9 TL074D

Commit message: Updated to resonance voltage control
Parts:
- added C25, C26, C27, C28, C29, C30, C31, C32: 100n, rcl:C-USC0805K
- added D5, D6, D8: 5.1V, diode:ZENER-DIODESOT23
- added D7: 1N4001, GMSN:DIODESMA
- added RES-2, RES-3: PJ301_THONKICONN6, og-pj301_variations:PJ301_THONKICONN6
- C1, C15, C16, C17, C19, C2, C20, C21, C22, C3, C4, C5, C6, C7, C8, C9: device rcl:C-USC0603 -> rcl:C-USC0805K
- C10, C24: device rcl:C-USC0603 -> Pure VCF:GMSN_C-USC0805K
- C11: device rcl:C-USC0603 -> Pure VCF:GMSN_R-US_M0805
- D3, D4: value 1N5819HW -> 1N4001; device diode:DIODE-SOD123 -> GMSN:DIODESMA
- POWER: value (none) -> SMD
- R1, R4: device rcl:R-US_R0805 -> Pure VCF:GMSN_R-US_M0805
- R10, R11, R2, R23, R28, R29, R3, R31, R32, R34, R35, R57, R58, R59, R6, R61, R63, R64, R65, R66, R68, R7, R8: device resistor:R-US_R0603 -> Pure VCF:GMSN_R-US_M0805
- R12, R13, R14, R15, R16, R17, R18, R19, R20, R21, R22, R24, R25, R26, R27, R30, R33, R36, R37, R38, R39, R40, R41, R42, R43, R44, R45, R46, R47, R48, R49, R50, R51, R52, R53, R54: device rcl:R-US_R0603 -> Pure VCF:GMSN_R-US_M0805
- R5: device GMSN:R-US_R0805 -> Pure VCF:GMSN_R-US_M0805
- R70, R72: value 10k -> 100k; device GMSN:R-US_R0805 -> Pure VCF:GMSN_R-US_M0805
- R71: value 10k -> 100k
- R73, R74: value 5k -> 100k
- renumbered IN1POT to IN1LEVEL, IN1POT1 to IN2LEVEL, IN1POT2 to IN3LEVEL
Connections:
- removed net 10V1: IC9A.+IN, RES-1.3
- removed net N$20: D2.C, POWER.2
- new net -12V-P: D2.C, POWER.1, POWER.2
- new net N$91: D7.A, RES-3.3
- new net N$92: D7.C, R74.2
- new net N$93: D8.C, IC1D.-IN, R74.1
- net -12V: now also C26.2, C28.2, C30.2, C32.2
- net 10V: no longer R69.2
- net 12V: now also C25.1, C27.1, C29.1, C31.1
- net 5V: now also R69.2, R71.2, R73.2
- net GND: now also C25.2, C26.1, C27.2, C28.1, C29.2, C30.1, C31.2, C32.1, D5.A, D6.A, D8.A, RES-2.1, RES-3.1; no longer IC9C.+IN, IC9D.+IN
- net N$6: now also POWER.9
- net N$78: now also D3.A, RES-2.3; no longer POWER.1
- net N$85: now also D3.C; no longer IC9A.-IN, IC9A.OUT, R70.1
- net N$86: now also D4.A, RES-1.3; no longer D3.C, IC9C.-IN, R70.2, R71.2
- net N$87: now also R70.2; no longer D3.A, IC9C.OUT
- net N$88: now also D5.C, IC9A.+IN, R70.1; no longer D4.A, R71.1, R73.2
- net N$89: now also D6.C, IC9C.+IN; no longer IC9D.-IN, R73.1, R74.2
- net N$9: now also R71.1, RES-2.2; no longer POWER.9
- net N$90: now also R73.1, RES-3.2; no longer IC9D.OUT, R74.1
- net RESONANCE_IN1: now also IC9A.-IN, IC9A.OUT
- net RESONANCE_IN2: now also IC9C.-IN, IC9C.OUT
- net RESONANCE_IN3: now also IC1D.+IN, IC1D.OUT
Other:
- moved on the sheet: C1, C13, C14, C2, C3, C4, C5, C6, D3, D4, IC9A, IC9C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

Commit message: fixed resonance input routing
Connections:
- new net RESONANCE_CTL1: R25.2, R4-RES1.S
- new net RESONANCE_CTL2: R39.2, R55-RES2.S
- new net RESONANCE_CTL3: R51.2, R56-RES3.S
- net 5V: no longer R4-RES1.E, R55-RES2.E, R56-RES3.E
- net RESONANCE_IN1: now also R4-RES1.E; no longer R25.2, R4-RES1.S
- net RESONANCE_IN2: now also R55-RES2.E; no longer R39.2, R55-RES2.S
- net RESONANCE_IN3: now also R56-RES3.E; no longer R51.2, R56-RES3.S
Other:
- moved on the sheet: D4, IC9A, R69, RES-1
